Commit message: Updated Bot Description

File: duke_bot_description/urdf/duke_bot.xacro (robot description, xacro)
@@ -126,50 +126,50 @@
 <link name="motor_holder_1_1">
   <inertial>
-    <origin xyz="0.007893675764047878 -0.003299542409627494 0.006737399954877261" rpy="0 0 0"/>
+    <origin xyz="-0.008486420552512978 0.0010897278578822153 -0.006738007055746277" rpy="0 0 0"/>
+    <mass value="0.0005943127590983897"/>
+    <inertia ixx="0.0" iyy="0.0" izz="0.0" ixy="0.0" iyz="-0.0" ixz="-0.0"/>
+  </inertial>
+  <visual>
+    <origin xyz="-0.022406 -0.046059 -0.000783" rpy="0 0 0"/>
+    <geometry>
+      <mesh filename="file://$(find duke_bot_description)/meshes/motor_holder_1_1.stl" scale="0.001 0.001 0.001"/>
+    </geometry>
+    <material name="silver"/>
+  </visual>
+  <collision>
+    <origin xyz="-0.022406 -0.046059 -0.000783" rpy="0 0 0"/>
+    <geometry>
+      <mesh filename="file://$(find duke_bot_description)/meshes/motor_holder_1_1.stl" scale="0.001 0.001 0.001"/>
+    </geometry>
+  </collision>
+</link>
+<link name="motor_holder_2_1">
+  <inertial>
+    <origin xyz="0.003299502174232416 -0.007893715999442892 -0.006738007055746277" rpy="0 0 0"/>
     <mass value="0.0005943127590983897"/>
     <inertia ixx="0.0" iyy="0.0" izz="0.0" ixy="0.0" iyz="0.0" ixz="0.0"/>
   </inertial>
   <visual>
-    <origin xyz="-0.006076 -0.050632 -0.004783" rpy="0 0 0"/>
-    <geometry>
-      <mesh filename="file://$(find duke_bot_description)/meshes/motor_holder_1_1.stl" scale="0.001 0.001 0.001"/>
-    </geometry>
-    <material name="silver"/>
-  </visual>
-  <collision>
-    <origin xyz="-0.006076 -0.050632 -0.004783" rpy="0 0 0"/>
-    <geometry>
-      <mesh filename="file://$(find duke_bot_description)/meshes/motor_holder_1_1.stl" scale="0.001 0.001 0.001"/>
-    </geometry>
-  </collision>
-</link>
-<link name="motor_holder_2_1">
-  <inertial>
-    <origin xyz="-0.0010897680932773143 0.008486380317117933 0.006737399954877258" rpy="0 0 0"/>
+    <origin xyz="0.050213 0.005657 -0.000783" rpy="0 0 0"/>
+    <geometry>
+      <mesh filename="file://$(find duke_bot_description)/meshes/motor_holder_2_1.stl" scale="0.001 0.001 0.001"/>
+    </geometry>
+    <material name="silver"/>
+  </visual>
+  <collision>
+    <origin xyz="0.050213 0.005657 -0.000783" rpy="0 0 0"/>
+    <geometry>
+      <mesh filename="file://$(find duke_bot_description)/meshes/motor_holder_2_1.stl" scale="0.001 0.001 0.001"/>
+    </geometry>
+  </collision>
+</link>
+<link name="motor_holder_3_1">
+  <inertial>
+    <origin xyz="-0.005186966469112084 -0.006804034087772862 -0.006738007055746281" rpy="0 0 0"/>
     <mass value="0.0005943127590983897"/>
-    <inertia ixx="0.0" iyy="0.0" izz="0.0" ixy="0.0" iyz="-0.0" ixz="-0.0"/>
-  </inertial>
-  <visual>
-    <origin xyz="0.04564 0.021987 -0.004783" rpy="0 0 0"/>
-    <geometry>
-      <mesh filename="file://$(find duke_bot_description)/meshes/motor_holder_2_1.stl" scale="0.001 0.001 0.001"/>
-    </geometry>
-    <material name="silver"/>
-  </visual>
-  <collision>
-    <origin xyz="0.04564 0.021987 -0.004783" rpy="0 0 0"/>
-    <geometry>
-      <mesh filename="file://$(find duke_bot_description)/meshes/motor_holder_2_1.stl" scale="0.001 0.001 0.001"/>
-    </geometry>
-  </collision>
-</link>
-<link name="motor_holder_3_1">
-  <inertial>
-    <origin xyz="0.0068039938523777425 0.005186926233717422 0.006737399954877263" rpy="0 0 0"/>
-    <mass value="0.0005943127590983897"/>
-    <inertia ixx="0.0" iyy="0.0" izz="0.0" ixy="-0.0" iyz="0.0" ixz="-0.0"/>
-  </inertial>
-  <visual>
-    <origin xyz="-0.028313 0.039813 -0.004783" rpy="0 0 0"/>
+    <inertia ixx="0.0" iyy="0.0" izz="0.0" ixy="-0.0" iyz="-0.0" ixz="0.0"/>
+  </inertial>
+  <visual>
+    <origin xyz="-0.040232 0.027894 -0.000783" rpy="0 0 0"/>
     <geometry>
       <mesh filename="file://$(find duke_bot_description)/meshes/motor_holder_3_1.stl" scale="0.001 0.001 0.001"/>
@@ -178,5 +178,5 @@
   </visual>
   <collision>
-    <origin xyz="-0.028313 0.039813 -0.004783" rpy="0 0 0"/>
+    <origin xyz="-0.040232 0.027894 -0.000783" rpy="0 0 0"/>
     <geometry>
       <mesh filename="file://$(find duke_bot_description)/meshes/motor_holder_3_1.stl" scale="0.001 0.001 0.001"/>
@@ -186,10 +186,10 @@
 <link name="n20_motor_1_1">
   <inertial>
-    <origin xyz="0.0008171801610878486 0.0029516368492447653 -0.004981275256068623" rpy="0 0 0"/>
+    <origin xyz="0.0007687298639330025 0.0029638635268054714 0.004980668155199606" rpy="0 0 0"/>
     <mass value="0.017834183296614247"/>
-    <inertia ixx="1e-06" iyy="0.0" izz="1e-06" ixy="-0.0" iyz="-0.0" ixz="0.0"/>
-  </inertial>
-  <visual>
-    <origin xyz="-0.013877 -0.046988 -0.016783" rpy="0 0 0"/>
+    <inertia ixx="1e-06" iyy="0.0" izz="1e-06" ixy="-0.0" iyz="0.0" ixz="0.0"/>
+  </inertial>
+  <visual>
+    <origin xyz="-0.013827 -0.046805 0.011217" rpy="0 0 0"/>
     <geometry>
       <mesh filename="file://$(find duke_bot_description)/meshes/n20_motor_1_1.stl" scale="0.001 0.001 0.001"/>
@@ -198,5 +198,5 @@
   </visual>
   <collision>
-    <origin xyz="-0.013877 -0.046988 -0.016783" rpy="0 0 0"/>
+    <origin xyz="-0.013827 -0.046805 0.011217" rpy="0 0 0"/>
     <geometry>
       <mesh filename="file://$(find duke_bot_description)/meshes/n20_motor_1_1.stl" scale="0.001 0.001 0.001"/>
@@ -206,10 +206,10 @@
 <link name="n20_motor_2_1">
   <inertial>
-    <origin xyz="-0.0029639037622005635 -0.0007687700993280529 -0.00498127525606863" rpy="0 0 0"/>
+    <origin xyz="-0.0029516770846398296 -0.000816220396482872 0.0049806681551996124" rpy="0 0 0"/>
     <mass value="0.017834183296614247"/>
-    <inertia ixx="0.0" iyy="1e-06" izz="1e-06" ixy="-0.0" iyz="0.0" ixz="0.0"/>
-  </inertial>
-  <visual>
-    <origin xyz="0.046386 0.013408 -0.016783" rpy="0 0 0"/>
+    <inertia ixx="0.0" iyy="1e-06" izz="1e-06" ixy="-0.0" iyz="0.0" ixz="-0.0"/>
+  </inertial>
+  <visual>
+    <origin xyz="0.046569 0.013459 0.011217" rpy="0 0 0"/>
     <geometry>
       <mesh filename="file://$(find duke_bot_description)/meshes/n20_motor_2_1.stl" scale="0.001 0.001 0.001"/>
@@ -218,5 +218,5 @@
   </visual>
   <collision>
-    <origin xyz="0.046386 0.013408 -0.016783" rpy="0 0 0"/>
+    <origin xyz="0.046569 0.013459 0.011217" rpy="0 0 0"/>
     <geometry>
       <mesh filename="file://$(find duke_bot_description)/meshes/n20_motor_2_1.stl" scale="0.001 0.001 0.001"/>
@@ -226,10 +226,10 @@
 <link name="n20_motor_3_1">
   <inertial>
-    <origin xyz="0.0021828842993763253 -0.002147566642738158 -0.005019331844800388" rpy="0 0 0"/>
+    <origin xyz="0.002147526407343482 -0.0021829245347714382 0.005018724743931371" rpy="0 0 0"/>
     <mass value="0.017834183296614247"/>
     <inertia ixx="1e-06" iyy="1e-06" izz="1e-06" ixy="0.0" iyz="-0.0" ixz="-0.0"/>
   </inertial>
   <visual>
-    <origin xyz="-0.035369 0.034878 -0.016783" rpy="0 0 0"/>
+    <origin xyz="-0.035297 0.03495 0.011217" rpy="0 0 0"/>
     <geometry>
       <mesh filename="file://$(find duke_bot_description)/meshes/n20_motor_3_1.stl" scale="0.001 0.001 0.001"/>
@@ -238,5 +238,5 @@
   </visual>
   <collision>
-    <origin xyz="-0.035369 0.034878 -0.016783" rpy="0 0 0"/>
+    <origin xyz="-0.035297 0.03495 0.011217" rpy="0 0 0"/>
     <geometry>
       <mesh filename="file://$(find duke_bot_description)/meshes/n20_motor_3_1.stl" scale="0.001 0.001 0.001"/>
@@ -244,363 +244,90 @@
   </collision>
 </link>
-<link name="omni_wheel_rim_1_1">
-  <inertial>
-    <origin xyz="-0.0009220541415564561 -0.0034401940247394402 -3.0355043873636633e-07" rpy="0 0 0"/>
-    <mass value="0.004947964863035424"/>
-    <inertia ixx="0.0" iyy="1e-06" izz="0.0" ixy="0.0" iyz="-0.0" ixz="0.0"/>
-  </inertial>
-  <visual>
-    <origin xyz="-0.02128 -0.074614 -0.011783" rpy="0 0 0"/>
-    <geometry>
-      <mesh filename="file://$(find duke_bot_description)/meshes/omni_wheel_rim_1_1.stl" scale="0.001 0.001 0.001"/>
-    </geometry>
-    <material name="silver"/>
-  </visual>
-  <collision>
-    <origin xyz="-0.02128 -0.074614 -0.011783" rpy="0 0 0"/>
-    <geometry>
-      <mesh filename="file://$(find duke_bot_description)/meshes/omni_wheel_rim_1_1.stl" scale="0.001 0.001 0.001"/>
-    </geometry>
-  </collision>
-</link>
-<link name="omni_wheel_rim_2_1">
-  <inertial>
-    <origin xyz="0.00343988349773669 0.0009221103126569735 -3.0355043874330523e-07" rpy="0 0 0"/>
-    <mass value="0.004947964863035424"/>
-    <inertia ixx="1e-06" iyy="0.0" izz="0.0" ixy="0.0" iyz="0.0" ixz="-0.0"/>
-  </inertial>
-  <visual>
-    <origin xyz="0.074011 0.020811 -0.011783" rpy="0 0 0"/>
-    <geometry>
-      <mesh filename="file://$(find duke_bot_description)/meshes/omni_wheel_rim_2_1.stl" scale="0.001 0.001 0.001"/>
-    </geometry>
-    <material name="silver"/>
-  </visual>
-  <collision>
-    <origin xyz="0.074011 0.020811 -0.011783" rpy="0 0 0"/>
-    <geometry>
-      <mesh filename="file://$(find duke_bot_description)/meshes/omni_wheel_rim_2_1.stl" scale="0.001 0.001 0.001"/>
-    </geometry>
-  </collision>
-</link>
-<link name="omni_wheel_rim_3_1">
-  <inertial>
-    <origin xyz="-0.002518066162622845 0.0025179863145547918 -3.035504302813241e-07" rpy="0 0 0"/>
-    <mass value="0.004947964863035424"/>
-    <inertia ixx="1e-06" iyy="1e-06" izz="0.0" ixy="-0.0" iyz="-0.0" ixz="-0.0"/>
-  </inertial>
-  <visual>
-    <origin xyz="-0.055592 0.055101 -0.011783" rpy="0 0 0"/>
-    <geometry>
-      <mesh filename="file://$(find duke_bot_description)/meshes/omni_wheel_rim_3_1.stl" scale="0.001 0.001 0.001"/>
-    </geometry>
-    <material name="silver"/>
-  </visual>
-  <collision>
-    <origin xyz="-0.055592 0.055101 -0.011783" rpy="0 0 0"/>
-    <geometry>
-      <mesh filename="file://$(find duke_bot_description)/meshes/omni_wheel_rim_3_1.stl" scale="0.001 0.001 0.001"/>
-    </geometry>
-  </collision>
-</link>
-<link name="wheel1_beadsa_1">
-  <inertial>
-    <origin xyz="0.002307677064762023 -0.008612699272992023 -0.0028975172251801615" rpy="0 0 0"/>
-    <mass value="0.0007686151878187868"/>
-    <inertia ixx="0.0" iyy="0.0" izz="0.0" ixy="0.0" iyz="-0.0" ixz="0.0"/>
-  </inertial>
-  <visual>
-    <origin xyz="0.071588 0.016089 -0.030016" rpy="0 0 0"/>
-    <geometry>
-      <mesh filename="file://$(find duke_bot_description)/meshes/wheel1_beadsa_1.stl" scale="0.001 0.001 0.001"/>
-    </geometry>
-    <material name="silver"/>
-  </visual>
-  <collision>
-    <origin xyz="0.071588 0.016089 -0.030016" rpy="0 0 0"/>
-    <geometry>
-      <mesh filename="file://$(find duke_bot_description)/meshes/wheel1_beadsa_1.stl" scale="0.001 0.001 0.001"/>
-    </geometry>
-  </collision>
-</link>
-<link name="wheel1_beadsb_1">
-  <inertial>
-    <origin xyz="0.0014266101738266285 -0.0053227005645062 0.007584733642780124" rpy="0 0 0"/>
-    <mass value="0.0007686151878187868"/>
+<link name="omni_wheel_1_1">
+  <inertial>
+    <origin xyz="-0.0009107726794966298 -0.0033974504948327405 -3.027244888445524e-07" rpy="0 0 0"/>
+    <mass value="0.007322790160921375"/>
+    <inertia ixx="1e-06" iyy="1e-06" izz="1e-06" ixy="0.0" iyz="0.0" ixz="-0.0"/>
+  </inertial>
+  <visual>
+    <origin xyz="-0.02123 -0.07443 0.006217" rpy="0 0 0"/>
+    <geometry>
+      <mesh filename="file://$(find duke_bot_description)/meshes/omni_wheel_1_1.stl" scale="0.001 0.001 0.001"/>
+    </geometry>
+    <material name="silver"/>
+  </visual>
+  <collision>
+    <origin xyz="-0.02123 -0.07443 0.006217" rpy="0 0 0"/>
+    <geometry>
+      <mesh filename="file://$(find duke_bot_description)/meshes/omni_wheel_1_1.stl" scale="0.001 0.001 0.001"/>
+    </geometry>
+  </collision>
+</link>
+<link name="omni_wheel_2_1">
+  <inertial>
+    <origin xyz="0.0033976805510785163 0.0009106360374820689 -3.043763801635971e-07" rpy="0 0 0"/>
+    <mass value="0.007322790160921375"/>
+    <inertia ixx="1e-06" iyy="1e-06" izz="1e-06" ixy="0.0" iyz="-0.0" ixz="0.0"/>
+  </inertial>
+  <visual>
+    <origin xyz="0.074195 0.020861 0.006217" rpy="0 0 0"/>
+    <geometry>
+      <mesh filename="file://$(find duke_bot_description)/meshes/omni_wheel_2_1.stl" scale="0.001 0.001 0.001"/>
+    </geometry>
+    <material name="silver"/>
+  </visual>
+  <collision>
+    <origin xyz="0.074195 0.020861 0.006217" rpy="0 0 0"/>
+    <geometry>
+      <mesh filename="file://$(find duke_bot_description)/meshes/omni_wheel_2_1.stl" scale="0.001 0.001 0.001"/>
+    </geometry>
+  </collision>
+</link>
+<link name="omni_wheel_3_1">
+  <inertial>
+    <origin xyz="-0.002486936407590054 0.0024869319581574886 -3.043763801679339e-07" rpy="0 0 0"/>
+    <mass value="0.007322790160921375"/>
+    <inertia ixx="1e-06" iyy="1e-06" izz="1e-06" ixy="-0.0" iyz="0.0" ixz="0.0"/>
+  </inertial>
+  <visual>
+    <origin xyz="-0.05552 0.055173 0.006217" rpy="0 0 0"/>
+    <geometry>
+      <mesh filename="file://$(find duke_bot_description)/meshes/omni_wheel_3_1.stl" scale="0.001 0.001 0.001"/>
+    </geometry>
+    <material name="silver"/>
+  </visual>
+  <collision>
+    <origin xyz="-0.05552 0.055173 0.006217" rpy="0 0 0"/>
+    <geometry>
+      <mesh filename="file://$(find duke_bot_description)/meshes/omni_wheel_3_1.stl" scale="0.001 0.001 0.001"/>
+    </geometry>
+  </collision>
+</link>
+<link name="ov_camera_1">
+  <inertial>
+    <origin xyz="-0.0022579398219568503 0.002951945188588923 0.01554416229830156" rpy="0 0 0"/>
+    <mass value="0.0027092205032529094"/>
     <inertia ixx="0.0" iyy="0.0" izz="0.0" ixy="0.0" iyz="0.0" ixz="-0.0"/>
   </inertial>
   <visual>
-    <origin xyz="0.075373 0.001965 -0.013676" rpy="0 0 0"/>
-    <geometry>
-      <mesh filename="file://$(find duke_bot_description)/meshes/wheel1_beadsb_1.stl" scale="0.001 0.001 0.001"/>
-    </geometry>
-    <material name="silver"/>
-  </visual>
-  <collision>
-    <origin xyz="0.075373 0.001965 -0.013676" rpy="0 0 0"/>
-    <geometry>
-      <mesh filename="file://$(find duke_bot_description)/meshes/wheel1_beadsb_1.stl" scale="0.001 0.001 0.001"/>
-    </geometry>
-  </collision>
-</link>
-<link name="wheel1_beadsc_1">
-  <inertial>
-    <origin xyz="-0.00142638982617245 0.0053222994354902246 0.0075846592563574835" rpy="0 0 0"/>
-    <mass value="0.0007686151878187868"/>
-    <inertia ixx="0.0" iyy="0.0" izz="0.0" ixy="0.0" iyz="-0.0" ixz="0.0"/>
-  </inertial>
-  <visual>
-    <origin xyz="0.07252 0.01261 0.00528" rpy="0 0 0"/>
-    <geometry>
-      <mesh filename="file://$(find duke_bot_description)/meshes/wheel1_beadsc_1.stl" scale="0.001 0.001 0.001"/>
-    </geometry>
-    <material name="silver"/>
-  </visual>
-  <collision>
-    <origin xyz="0.07252 0.01261 0.00528" rpy="0 0 0"/>
-    <geometry>
-      <mesh filename="file://$(find duke_bot_description)/meshes/wheel1_beadsc_1.stl" scale="0.001 0.001 0.001"/>
-    </geometry>
-  </collision>
-</link>
-<link name="wheel1_beadsd_1">
-  <inertial>
-    <origin xyz="-0.002307322935239303 0.00861230072701295 -0.002897089875683309" rpy="0 0 0"/>
-    <mass value="0.0007686151878187868"/>
+    <origin xyz="0.022096 -0.022515 -0.004783" rpy="0 0 0"/>
+    <geometry>
+      <mesh filename="file://$(find duke_bot_description)/meshes/ov_camera_1.stl" scale="0.001 0.001 0.001"/>
+    </geometry>
+    <material name="silver"/>
+  </visual>
+  <collision>
+    <origin xyz="0.022096 -0.022515 -0.004783" rpy="0 0 0"/>
+    <geometry>
+      <mesh filename="file://$(find duke_bot_description)/meshes/ov_camera_1.stl" scale="0.001 0.001 0.001"/>
+    </geometry>
+  </collision>
+</link>
+<link name="fake_camera_1">
+  <inertial>
+    <origin xyz="-0.0022579398219568503 0.002951945188588923 0.01554416229830156" rpy="0 0 0"/>
+    <mass value="0.0027092205032529094"/>
     <inertia ixx="0.0" iyy="0.0" izz="0.0" ixy="0.0" iyz="0.0" ixz="-0.0"/>
   </inertial>
-  <visual>
-    <origin xyz="0.066973 0.033314 0.000656" rpy="0 0 0"/>
-    <geometry>
-      <mesh filename="file://$(find duke_bot_description)/meshes/wheel1_beadsd_1.stl" scale="0.001 0.001 0.001"/>
-    </geometry>
-    <material name="silver"/>
-  </visual>
-  <collision>
-    <origin xyz="0.066973 0.033314 0.000656" rpy="0 0 0"/>
-    <geometry>
-      <mesh filename="file://$(find duke_bot_description)/meshes/wheel1_beadsd_1.stl" scale="0.001 0.001 0.001"/>
-    </geometry>
-  </collision>
-</link>
-<link name="wheel1_beadse_1">
-  <inertial>
-    <origin xyz="4.6499714258241287e-07 -1.4235487700436922e-07 -0.00937530355043611" rpy="0 0 0"/>
-    <mass value="0.0007686151878187868"/>
-    <inertia ixx="0.0" iyy="0.0" izz="0.0" ixy="0.0" iyz="0.0" ixz="-0.0"/>
-  </inertial>
-  <visual>
-    <origin xyz="0.066397 0.035464 -0.021158" rpy="0 0 0"/>
-    <geometry>
-      <mesh filename="file://$(find duke_bot_description)/meshes/wheel1_beadse_1.stl" scale="0.001 0.001 0.001"/>
-    </geometry>
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
Commit message: feat: changed hdr wheel controller
Signed-off-by: Hari Vikinesh <harivikinesh@gmail.com>

File: duke_bot_description/urdf/duke_bot.xacro (robot description, xacro)
@@ -1,7 +1,11 @@
 <?xml version="1.0" ?>
 <robot name="duke_bot" xmlns:xacro="http://www.ros.org/wiki/xacro">
-<xacro:include filename="$(find duke_bot_description)/urdf/materials.xacro" />
-<xacro:include filename="$(find duke_bot_description)/urdf/duke_bot.trans" />
 <xacro:include filename="$(find duke_bot_description)/urdf/duke_bot.gazebo" />
+<link name ="footprint_link" />
+<joint name="footprint_joint" type="fixed">
+  <origin xyz="0.0 0.0 0.0" rpy="0 0 1.047" />
+  <parent link="footprint_link"/>
+  <child link="base_link"/>
+</joint>
 <link name="base_link">
   <inertial>
@@ -391,4 +395,5 @@
   <child link="omni_wheel_1_1"/>
   <axis xyz="0.258819 0.965926 -0.0"/>
+  <limit effort="5" velocity="5" />
 </joint>
 <joint name="wheel2_joint" type="continuous">
@@ -397,4 +402,5 @@
   <child link="omni_wheel_2_1"/>
   <axis xyz="-0.965926 -0.258819 -0.0"/>
+  <limit effort="5" velocity="5" />
 </joint>
 <joint name="wheel3_joint" type="continuous">
@@ -403,4 +409,5 @@
   <child link="omni_wheel_3_1"/>
   <axis xyz="0.707107 -0.707107 0.0"/>
+  <limit effort="5" velocity="5" />
 </joint>
 <joint name="camera_fix" type="fixed">
